File: schematic/irobot virtualwall.brd (EAGLE design)
At the start: 38.1 x 22.5 mm, 8 parts, among them IC1 TINY12P

Commit message: update
Parts:
- renumbered LED1 to IR_LED1
Changed lines of the file:
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@@
 <attribute name="VALUE" x="19.3294" y="1.905" size="1.27" layer="27" ratio="10"/>
 </element>
-<element name="LED1" library="led" library_urn="urn:adsk.eagle:library:259" package="LED5MM" package3d_urn="urn:adsk.eagle:package:15799/2" value="" x="39.37" y="17.78" smashed="yes" rot="R270">
+<element name="IR_LED1" library="led" library_urn="urn:adsk.eagle:library:259" package="LED5MM" package3d_urn="urn:adsk.eagle:package:15799/2" value="" x="39.37" y="17.78" smashed="yes" rot="R270">
 <attribute name="NAME" x="39.9034" y="14.605" size="1.27" layer="25" ratio="10" rot="R270"/>
 <attribute name="POPULARITY" value="93" x="39.37" y="17.78" size="1.778" layer="27" rot="R270" display="off"/>
@@
 <contactref element="IC1" pad="4"/>
 <contactref element="PAD2" pad="1"/>
-<contactref element="LED1" pad="K"/>
+<contactref element="IR_LED1" pad="K"/>
 <contactref element="LED2" pad="K"/>
 <wire x1="39.37" y1="16.51" x2="39.37" y2="5.08" width="0.4064" layer="16"/>
@@
 <signal name="N$3">
 <contactref element="R1" pad="2"/>
-<contactref element="LED1" pad="A"/>
+<contactref element="IR_LED1" pad="A"/>
 <wire x1="37.7825" y1="6.35" x2="26.67" y2="6.35" width="0.4064" layer="16"/>
 <wire x1="37.7825" y1="17.4625" x2="37.7825" y2="6.35" width="0.4064" layer="16"/>
