File: schematic/irobot virtualwall.sch (EAGLE design)
At the start: 8 parts, among them IC1 TINY12P

Commit message: update
Parts:
- renumbered LED1 to IR_LED1
Changed lines of the file:
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@@
 <part name="R1" library="rcl" library_urn="urn:adsk.eagle:library:334" deviceset="R-EU_" device="0207/10" package3d_urn="urn:adsk.eagle:package:23491/2"/>
 <part name="R2" library="rcl" library_urn="urn:adsk.eagle:library:334" deviceset="R-EU_" device="0207/10" package3d_urn="urn:adsk.eagle:package:23491/2"/>
-<part name="LED1" library="led" library_urn="urn:adsk.eagle:library:259" deviceset="LED" device="5MM" package3d_urn="urn:adsk.eagle:package:15799/2"/>
+<part name="IR_LED1" library="led" library_urn="urn:adsk.eagle:library:259" deviceset="LED" device="5MM" package3d_urn="urn:adsk.eagle:package:15799/2"/>
 <part name="LED2" library="led" library_urn="urn:adsk.eagle:library:259" deviceset="LED" device="5MM" package3d_urn="urn:adsk.eagle:package:15799/2"/>
 <part name="GND1" library="supply1" library_urn="urn:adsk.eagle:library:371" deviceset="GND" device=""/>
@@
 <attribute name="VALUE" x="95.25" y="32.258" size="1.778" layer="96"/>
 </instance>
-<instance part="LED1" gate="G$1" x="114.3" y="50.8" smashed="yes" rot="R90">
+<instance part="IR_LED1" gate="G$1" x="114.3" y="50.8" smashed="yes" rot="R90">
 <attribute name="NAME" x="118.872" y="54.356" size="1.778" layer="95" rot="R180"/>
 <attribute name="VALUE" x="118.872" y="56.515" size="1.778" layer="96" rot="R180"/>
@@
 </segment>
 <segment>
-<pinref part="LED1" gate="G$1" pin="C"/>
+<pinref part="IR_LED1" gate="G$1" pin="C"/>
 <pinref part="GND1" gate="1" pin="GND"/>
 <wire x1="119.38" y1="50.8" x2="124.46" y2="50.8" width="0.1524" layer="91"/>
@@
 <segment>
 <pinref part="R1" gate="G$1" pin="2"/>
-<pinref part="LED1" gate="G$1" pin="A"/>
+<pinref part="IR_LED1" gate="G$1" pin="A"/>
 <wire x1="104.14" y1="40.64" x2="104.14" y2="50.8" width="0.1524" layer="91"/>
 <wire x1="104.14" y1="50.8" x2="111.76" y2="50.8" width="0.1524" layer="91"/>
